File: nano_original_v3/nano_original.kicad_sch (KiCad schematic)
At the start: 32 parts, among them J1 USB_B_Micro, J2 Conn_01x15, J3 Conn_01x15, J4 Conn_02x03_Odd_Even, SW1 SW_Push, U1 LM1117MP-5.0, U2 FT231XS, U3 ATmega328P-M, Y1 16MHz

Commit message: updated BOM
Parts:
- J2, J3: footprint Connector_PinSocket_2.54mm:PinSocket_1x15_P2.54mm_Vertical -> Connector_PinHeader_2.54mm:PinHeader_1x15_P2.54mm_Vertical
- SW1: footprint Button_Switch_SMD:SW_Push_SPST_NO_Alps_SKRK -> Button_Switch_SMD:SW_SPST_B3U-1000P
- U3: value ATmega328P-M -> ATmega328P-MUR
Changed lines of the file:
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@@
 			)
 		)
-		(property "Footprint" "Connector_PinSocket_2.54mm:PinSocket_1x15_P2.54mm_Vertical"
+		(property "Footprint" "Connector_PinHeader_2.54mm:PinHeader_1x15_P2.54mm_Vertical"
 			(at 71.12 41.91 0)
 			(effects
@@
 			)
 		)
-		(property "Footprint" "Connector_PinSocket_2.54mm:PinSocket_1x15_P2.54mm_Vertical"
+		(property "Footprint" "Connector_PinHeader_2.54mm:PinHeader_1x15_P2.54mm_Vertical"
 			(at 41.91 41.91 0)
 			(effects
@@
 			)
 		)
-		(property "Footprint" "Button_Switch_SMD:SW_Push_SPST_NO_Alps_SKRK"
+		(property "Footprint" "Button_Switch_SMD:SW_SPST_B3U-1000P"
 			(at 130.81 38.1 0)
 			(effects
@@
 			)
 		)
-		(property "Value" "ATmega328P-M"
+		(property "Value" "ATmega328P-MUR"
 			(at 222.504 156.464 0)
 			(effects
